File: Fuel_System.kicad_sch (KiCad schematic)
At the start: 0 parts

Commit message: Added motorcontroll Added ignition, injector and start motor connectors
Parts:
- added D?: SM_On, symbol Device:LED_Small
- added D?: INJ_1, symbol Device:LED_Small
- added D?: 1N5820G, symbol Device:D_Small
- added D?: INJ_2, symbol Device:LED_Small
- added F? (x2): 5A, symbol Device:Fuse_Small
- added J?: IGN_2_Out, symbol Connector_Generic:Conn_01x03
- added J?: INJ_1_Out, symbol Connector_Generic:Conn_01x02
- added J?: SM_Conn., symbol Connector_Generic:Conn_01x02
- added J?: IGN_1_Out, symbol Connector_Generic:Conn_01x03
- added J?: INJ_2_Out, symbol Connector_Generic:Conn_01x02
- added R? (x3): 1k, symbol Device:R_Small
Connections:
- new net: D?.2 (A), R?.2 (x3)
- new net: F?.2, J?.2 (Pin_2), R?.1 (x2)
- new net +12V: D?.1 (K), J?.1 (Pin_1), J?.1 (Pin_1)
- new net Dead_Mans_Voltage: F?.1, F?.1
- new net GNDPWR: D?.1 (K), D?.1 (K), D?.1 (K), D?.2 (A), J?.2 (Pin_2), J?.3 (Pin_3), J?.3 (Pin_3)
- new net INJ_1: J?.1 (Pin_1)
- new net INJ_2: J?.1 (Pin_1)
- new net SPK_A_(IGN1): J?.2 (Pin_2)
- new net SPK_B_(IGN2): J?.2 (Pin_2)
- new net Start_Motor_Voltage: J?.1 (Pin_1), R?.1
Other:
- note added: "Fuel and Ignition system"
- note added: "Ignition 1 and 2 Conn."
- note added: "Injector 1 Conn."
- note added: "Injector 2 Conn."
- note added: "Not used in configuration for comp. 2023"
- note added: "SM = Start Motor Flywheel diode to prevent negative voltage"
- note added: "Start Motor Conn."
