File: Vera ECU 2.0.kicad_sch (KiCad schematic)
At the start: 35 parts

Commit message: Added relays
Added relays to the schematic and noted that a relay for the fuel injectors is not needed.
Parts:
- added D? (x2): 1N5820G, symbol Device:D_Small
- added K?: Start Motor Relay, symbol old-vera-ecu:Mini_ISO_relay
- added K?: Main Power Relay, symbol old-vera-ecu:Mini_ISO_relay
Connections:
- net Dead_Mans_Signal is gone; now on net Dead_Mans_Voltage: J?.5 (Pin_5)
- net +12V: now also K?.30, K?.87
- net +BATT: now also K?.30
- net GNDPWR: now also D?.2 (A), D?.2 (A), K?.85, K?.85
- net Main_Power_Signal: now also D?.1 (K), K?.86
- net Start_Motor_Signal: now also D?.1 (K), K?.86
- net Start_Motor_Voltage: now also K?.87
- no-connect marks 21 -> 23
Other:
- sheet Sensor connection notes renamed Sensor connection and other notes
- note added: "Battery is of type LiFePO4"
- note added: "For a (semi-)detailed description of the circuit, read this document about connections: https://docs.google.com/document/d/1L7XT-N4o6fV4hY6EBp9OTlTL3f0HpLTFqfsGH-qPXZ4/edit"
- note added: "Main Power Relay"
- note added: "Reference for Microsquirt connector: http://www.msextra.com/doc/pdf/Microsquirt_Hardware-3.3.pdf"
- note added: "Start Motor Relay"

Commit message: Changed position of flowback diode Changed the position of the diode for back current at the main power relay and start motor relay
Parts:
- removed D? (x2): 1N5820G, symbol Device:D_Small
- added D? (x2): 1N5820G, symbol Device:D_Small
Connections:
- net +12V: now also D?.1 (K)
- net +BATT: now also D?.1 (K)
- net GNDPWR: now also D?.2 (A), D?.2 (A)
Changed lines of the file:
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@@
   (junction (at 170.815 68.58) (diameter 0) (color 0 0 0 0)
   )
-  (junction (at 49.784 115.824) (diameter 0) (color 0 0 0 0)
-  )
-  (junction (at 70.358 115.824) (diameter 0) (color 0 0 0 0)
-  )
   (junction (at 143.002 64.262) (diameter 0) (color 0 0 0 0)
   )
@@
   (junction (at 268.478 37.846) (diameter 0) (color 0 0 0 0)
   )
+  (junction (at 78.74 125.984) (diameter 0) (color 0 0 0 0)
+  )
   (junction (at 235.585 41.91) (diameter 0) (color 0 0 0 0)
   )
   (junction (at 50.8 33.02) (diameter 0) (color 0 0 0 0)
   )
+  (junction (at 70.358 125.984) (diameter 0) (color 0 0 0 0)
+  )
   (junction (at 173.736 121.158) (diameter 0) (color 0 0 0 0)
   )
@@
   (junction (at 271.018 43.561) (diameter 0) (color 0 0 0 0)
   )
-  (junction (at 16.256 115.824) (diameter 0) (color 0 0 0 0)
+  (junction (at 24.638 125.984) (diameter 0) (color 0 0 0 0)
   )
   (junction (at 235.585 31.75) (diameter 0) (color 0 0 0 0)
   )
-  (junction (at 103.886 115.824) (diameter 0) (color 0 0 0 0)
+  (junction (at 16.256 125.984) (diameter 0) (color 0 0 0 0)
   )
   (junction (at 235.585 29.21) (diameter 0) (color 0 0 0 0)
@@
     (stroke (width 0) (type default) (color 0 0 0 0))
   )
-  (wire (pts (xy 101.6 115.824) (xy 103.886 115.824))
-    (stroke (width 0) (type default) (color 0 0 0 0))
-  )
   (wire (pts (xy 168.656 46.736) (xy 168.656 48.006))
     (stroke (width 0) (type default) (color 0 0 0 0))
@@
     (stroke (width 0) (type default) (color 0 0 0 0))
   )
-  (wire (pts (xy 49.784 115.824) (xy 51.816 115.824))
+  (wire (pts (xy 47.498 115.824) (xy 51.816 115.824))
     (stroke (width 0) (type default) (color 0 0 0 0))
   )
@@
     (stroke (width 0) (type default) (color 0 0 0 0))
   )
-  (wire (pts (xy 49.784 106.172) (xy 49.784 115.824))
-    (stroke (width 0) (type default) (color 0 0 0 0))
-  )
   (wire (pts (xy 52.07 81.28) (xy 52.07 78.74))
     (stroke (width 0) (type default) (color 0 0 0 0))
@@
     (stroke (width 0) (type default) (color 0 0 0 0))
   )
+  (wire (pts (xy 16.256 125.984) (xy 17.78 125.984))
+    (stroke (width 0) (type default) (color 0 0 0 0))
+  )
   (wire (pts (xy 50.8 24.13) (xy 50.8 25.4))
     (stroke (width 0) (type default) (color 0 0 0 0))
@@
     (stroke (width 0) (type default) (color 0 0 0 0))
   )
-  (wire (pts (xy 16.256 106.172) (xy 16.256 115.824))
-    (stroke (width 0) (type default) (color 0 0 0 0))
-  )
   (wire (pts (xy 143.002 75.692) (xy 143.002 71.882))
     (stroke (width 0) (type default) (color 0 0 0 0))
@@
     (stroke (width 0) (type default) (color 0 0 0 0))
   )
-  (wire (pts (xy 16.256 115.824) (xy 16.256 129.54))
+  (wire (pts (xy 16.256 115.824) (xy 16.256 125.984))
     (stroke (width 0) (type default) (color 0 0 0 0))
   )
@@
     (stroke (width 0) (type default) (color 0 0 0 0))
   )
-  (wire (pts (xy 34.798 106.172) (xy 16.256 106.172))
-    (stroke (width 0) (type default) (color 0 0 0 0))
-  )
   (wire (pts (xy 247.65 68.58) (xy 251.46 68.58))
     (stroke (width 0) (type default) (color 0 0 0 0))
@@
     (stroke (width 0) (type default) (color 0 0 0 0))
   )
-  (wire (pts (xy 70.358 106.172) (xy 70.358 115.824))
-    (stroke (width 0) (type default) (color 0 0 0 0))
-  )
   (wire (pts (xy 199.39 30.48) (xy 198.374 30.48))
     (stroke (width 0) (type default) (color 0 0 0 0))
@@
     (stroke (width 0) (type default) (color 0 0 0 0))
   )
+  (wire (pts (xy 70.358 125.984) (xy 70.358 133.35))
+    (stroke (width 0) (type default) (color 0 0 0 0))
+  )
   (wire (pts (xy 235.585 42.545) (xy 235.585 41.91))
     (stroke (width 0) (type default) (color 0 0 0 0))
@@
     (stroke (width 0) (type default) (color 0 0 0 0))
   )
-  (wire (pts (xy 88.9 106.172) (xy 70.358 106.172))
-    (stroke (width 0) (type default) (color 0 0 0 0))
-  )
   (wire (pts (xy 140.97 44.45) (xy 144.78 44.45))
     (stroke (width 0) (type default) (color 0 0 0 0))
   )
-  (wire (pts (xy 93.98 106.172) (xy 103.886 106.172))
-    (stroke (width 0) (type default) (color 0 0 0 0))
-  )
   (wire (pts (xy 209.55 63.5) (xy 209.55 62.23))
     (stroke (width 0) (type default) (color 0 0 0 0))
   )
-  (wire (pts (xy 70.358 115.824) (xy 70.358 133.35))
+  (wire (pts (xy 70.358 115.824) (xy 70.358 125.984))
     (stroke (width 0) (type default) (color 0 0 0 0))
   )
@@
     (stroke (width 0) (type default) (color 0 0 0 0))
   )
+  (wire (pts (xy 76.962 125.984) (xy 78.74 125.984))
+    (stroke (width 0) (type default) (color 0 0 0 0))
+  )
   (wire (pts (xy 78.74 123.952) (xy 78.74 125.984))
     (stroke (width 0) (type default) (color 0 0 0 0))
   )
-  (wire (pts (xy 47.498 115.824) (xy 49.784 115.824))
-    (stroke (width 0) (type default) (color 0 0 0 0))
-  )
-  (wire (pts (xy 39.878 106.172) (xy 49.784 106.172))
-    (stroke (width 0) (type default) (color 0 0 0 0))
-  )
   (wire (pts (xy 235.585 39.37) (xy 240.03 39.37))
     (stroke (width 0) (type default) (color 0 0 0 0))
@@
     (stroke (width 0) (type default) (color 0 0 0 0))
   )
-  (wire (pts (xy 103.886 115.824) (xy 105.918 115.824))
+  (wire (pts (xy 101.6 115.824) (xy 105.918 115.824))
     (stroke (width 0) (type default) (color 0 0 0 0))
   )
@@
     (stroke (width 0) (type default) (color 0 0 0 0))
   )
+  (wire (pts (xy 22.86 125.984) (xy 24.638 125.984))
+    (stroke (width 0) (type default) (color 0 0 0 0))
+  )
   (wire (pts (xy 87.63 35.56) (xy 88.9 35.56))
     (stroke (width 0) (type default) (color 0 0 0 0))
@@
     (stroke (width 0) (type default) (color 0 0 0 0))
   )
-  (wire (pts (xy 103.886 106.172) (xy 103.886 115.824))
-    (stroke (width 0) (type default) (color 0 0 0 0))
-  )
   (wire (pts (xy 143.764 132.334) (xy 146.304 132.334))
     (stroke (width 0) (type default) (color 0 0 0 0))
@@
     (stroke (width 0) (type default) (color 0 0 0 0))
   )
+  (wire (pts (xy 70.358 125.984) (xy 71.882 125.984))
+    (stroke (width 0) (type default) (color 0 0 0 0))
+  )
   (wire (pts (xy 136.652 61.722) (xy 137.922 61.722))
     (stroke (width 0) (type default) (color 0 0 0 0))
@@
   )
   (polyline (pts (xy 259.715 17.78) (xy 259.715 53.34))
+    (stroke (width 0) (type default) (color 0 0 0 0))
+  )
+  (wire (pts (xy 16.256 125.984) (xy 16.256 129.54))
     (stroke (width 0) (type default) (color 0 0 0 0))
   )
@@
     )
     (property "Datasheet" "~" (id 3) (at 50.8 27.94 0)
+      (effects (font (size 1.27 1.27)) hide)
+    )
+    (pin "1")
+    (pin "2")
+  )
+  (symbol (lib_id "Device:D_Small") (at 74.422 125.984 180) (unit 1)
+    (in_bom yes) (on_board yes)
+    (property "Reference" "D?" (id 0) (at 74.422 124.206 0))
+    (property "Value" "1N5820G" (id 1) (at 74.93 128.016 0))
+    (property "Footprint" "" (id 2) (at 74.422 125.984 90)
+      (effects (font (size 1.27 1.27)) hide)
+    )
+    (property "Datasheet" "~" (id 3) (at 74.422 125.984 90)
       (effects (font (size 1.27 1.27)) hide)
     )
@@
     )
     (pin "1")
+  )
+  (symbol (lib_id "Device:D_Small") (at 20.32 125.984 180) (unit 1)
+    (in_bom yes) (on_board yes)
+    (property "Reference" "D?" (id 0) (at 20.32 124.206 0))
+    (property "Value" "1N5820G" (id 1) (at 20.828 128.016 0))
+    (property "Footprint" "" (id 2) (at 20.32 125.984 90)
+      (effects (font (size 1.27 1.27)) hide)
+    )
+    (property "Datasheet" "~" (id 3) (at 20.32 125.984 90)
+      (effects (font (size 1.27 1.27)) hide)
+    )
+    (pin "1")
+    (pin "2")
   )
   (symbol (lib_id "power:GNDPWR") (at 137.922 75.692 0) (unit 1)
@@
     (pin "1")
   )
-  (symbol (lib_id "Device:D_Small") (at 91.44 106.172 180) (unit 1)
-    (in_bom yes) (on_board yes)
-    (property "Reference" "D?" (id 0) (at 91.44 104.394 0))
-    (property "Value" "1N5820G" (id 1) (at 91.44 108.204 0))
-    (property "Footprint" "" (id 2) (at 91.44 106.172 90)
-      (effects (font (size 1.27 1.27)) hide)
-    )
-    (property "Datasheet" "~" (id 3) (at 91.44 106.172 90)
-      (effects (font (size 1.27 1.27)) hide)
-    )
-    (pin "1")
-    (pin "2")
-  )
   (symbol (lib_id "power:+5V") (at 235.966 94.996 0) (unit 1)
     (in_bom yes) (on_board yes)
@@
     )
     (pin "1")
-  )
-  (symbol (lib_id "Device:D_Small") (at 37.338 106.172 180) (unit 1)
-    (in_bom yes) (on_board yes)
-    (property "Reference" "D?" (id 0) (at 37.338 104.394 0))
-    (property "Value" "1N5820G" (id 1) (at 37.338 108.204 0))
-    (property "Footprint" "" (id 2) (at 37.338 106.172 90)
-      (effects (font (size 1.27 1.27)) hide)
-    )
-    (property "Datasheet" "~" (id 3) (at 37.338 106.172 90)
-      (effects (font (size 1.27 1.27)) hide)
-    )
-    (pin "1")
-    (pin "2")
   )
   (symbol (lib_id "power:+12V") (at 143.764 119.634 0) (unit 1)
@@
       (reference "D?") (unit 1) (value "1N5820G") (footprint "")
     )
+    (path "/29fec646-b7b6-41d5-a2c5-540ff8224ace"
+      (reference "D?") (unit 1) (value "1N5820G") (footprint "")
+    )
     (path "/579ea284-ce75-49a0-93c9-816f19093dbf"
       (reference "D?") (unit 1) (value "Power_on") (footprint "")
     )
+    (path "/62106959-3ce1-474f-80f2-94a4c5d0b81a"
+      (reference "D?") (unit 1) (value "1N5820G") (footprint "")
+    )
     (path "/666c77af-0c34-4edd-a5ac-a05f1f9811eb"
       (reference "D?") (unit 1) (value "BKLGT_POW") (footprint "")
@@
       (reference "D?") (unit 1) (value "EGO Pre-warmer") (footprint "")
     )
-    (path "/a3625b4c-1e39-48ec-a83a-68094c1145dc"
-      (reference "D?") (unit 1) (value "1N5820G") (footprint "")
-    )
-    (path "/d00c4904-3e0f-478e-8b3e-affd00c8c035"
-      (reference "D?") (unit 1) (value "1N5820G") (footprint "")
-    )
     (path "/286984fe-7ba7-48af-88e9-b321ea325776"

Commit message: Added motorcontroll Added ignition, injector and start motor connectors
Parts:
- added D?: 1N5820G, symbol Device:D_Small
Connections:
- net +12V: now also D?.2 (A)
- net +BATT: now also D?.1 (K)
- net SMS_TO_RELAY: now also K?.86
- net Start_Motor_Signal: no longer K?.86
Other:
- note added: "Backlight Conn."
- note added: "Cockpit Conn."
- note added: "Diode to prevent negative voltage if fuse is burnt"
- note removed: "Backlight connection"
- note removed: "Cockpit connector"
